Commit message: [fix] everything runs as it is now!

File: data/avatar/urdf/panda_arm.urdf (robot description, URDF)
Before this commit: robot panda, 9 links, 8 joints
Links:
- link panda_link0: geometry collision sphere radius=0.06; collision sphere radius=0.06
- link panda_link1: geometry collision sphere radius=0.06; collision sphere radius=0.06
- link panda_link2: geometry collision sphere radius=0.06; collision sphere radius=0.06
- link panda_link3: geometry collision sphere radius=0.06; collision sphere radius=0.06
- link panda_link4: geometry collision sphere radius=0.05; collision sphere radius=0.055
- link panda_link5: geometry collision sphere radius=0.035; collision sphere radius=0.035
- link panda_link6: geometry collision sphere radius=0.04; collision sphere radius=0.04
- link panda_link7: geometry collision sphere radius=0.05; collision sphere radius=0.06
