Commit message: [phew] port to ros2, lot of ros related clean up and reorg

File: data/avatar/urdf/avatar_gripper_right.urdf (robot description, URDF)
Before this commit: robot avatar_gripper_3f_model, 13 links, 12 joints
Links:
- link right_gripper_base: geometry visual mesh filename=..meshes/right/gripper_base.obj
- link right_index_base_connector: geometry collision sphere radius=0.015; collision sphere radius=0.015
- link right_index_fingertip: geometry collision cylinder length=0.023 radius=0.008; collision cylinder length=0.026 radius=0.008
- link right_index_knuckle: geometry collision cylinder length=0.04 radius=0.01; collision sphere radius=0.01
- link right_middle_fingertip: geometry collision cylinder length=0.023 radius=0.008; collision cylinder length=0.026 radius=0.008
- link right_middle_knuckle: geometry collision cylinder length=0.04 radius=0.01; collision sphere radius=0.01
- link right_thumb_base: geometry collision cylinder length=0.036 radius=0.01; collision sphere radius=0.01
- link right_thumb_finger: geometry collision cylinder length=0.041 radius=0.008; collision sphere radius=0.008
- link right_thumb_knuckle: geometry collision cylinder length=0.047 radius=0.009; collision sphere radius=0.009
- link right_thumb_swivel_link: geometry visual mesh filename=..meshes/right/thumb_swivel_link.obj

File: data/avatar/urdf/avatar_gripper_right_nomimic.urdf (robot description, URDF)
Before this commit: robot avatar_gripper_3f_model, 13 links, 12 joints
Links:
- link right_gripper_base: geometry visual mesh filename=../meshes/right/gripper_base.obj
- link right_index_base_connector: geometry collision sphere radius=0.015; collision sphere radius=0.015
- link right_index_fingertip: geometry collision cylinder length=0.023 radius=0.008; collision cylinder length=0.026 radius=0.008
- link right_index_knuckle: geometry collision cylinder length=0.04 radius=0.01; collision sphere radius=0.01
- link right_middle_fingertip: geometry collision cylinder length=0.023 radius=0.008; collision cylinder length=0.026 radius=0.008
- link right_middle_knuckle: geometry collision cylinder length=0.04 radius=0.01; collision sphere radius=0.01
- link right_thumb_base: geometry collision cylinder length=0.036 radius=0.01; collision sphere radius=0.01
- link right_thumb_finger: geometry collision cylinder length=0.041 radius=0.008; collision sphere radius=0.008
- link right_thumb_knuckle: geometry collision cylinder length=0.047 radius=0.009; collision sphere radius=0.009
- link right_thumb_swivel_link: geometry visual mesh filename=../meshes/right/thumb_swivel_link.obj

File: data/avatar/urdf/panda_arm_avatar.urdf (robot description, URDF)
Before this commit: robot panda, 22 links, 21 joints
Links:
- link panda_hand: geometry visual mesh filename=../meshes/gripper_base.obj
- link panda_link0: geometry collision sphere radius=0.06; collision sphere radius=0.06
- link panda_link1: geometry collision sphere radius=0.06; collision sphere radius=0.06
- link panda_link2: geometry collision sphere radius=0.06; collision sphere radius=0.06
- link panda_link3: geometry collision sphere radius=0.06; collision sphere radius=0.06
- link panda_link4: geometry collision sphere radius=0.05; collision sphere radius=0.055
- link panda_link5: geometry collision sphere radius=0.035; collision sphere radius=0.035
- link panda_link6: geometry collision sphere radius=0.04; collision sphere radius=0.04
- link panda_link7: geometry collision sphere radius=0.05; collision sphere radius=0.06
- link right_index_base_connector: geometry visual mesh filename=../meshes/index_base_connector.obj
- link right_index_fingertip: geometry collision mesh filename=../meshes/index_fingertip.obj; visual mesh filename=../meshes/index_fingertip.obj
- link right_index_knuckle: geometry collision mesh filename=../meshes/index_knuckle.obj; visual mesh filename=../meshes/index_knuckle.obj
- link right_middle_fingertip: geometry collision mesh filename=../meshes/index_fingertip.obj; visual mesh filename=../meshes/index_fingertip.obj
- link right_middle_knuckle: geometry collision mesh filename=../meshes/index_knuckle.obj; visual mesh filename=../meshes/index_knuckle.obj
- link right_thumb_base: geometry collision mesh filename=../meshes/thumb_base_extra.obj; visual mesh filename=../meshes/thumb_base_extra.obj
- link right_thumb_finger: geometry collision mesh filename=../meshes/thumb_fingertip.obj; visual mesh filename=../meshes/thumb_fingertip.obj
- link right_thumb_knuckle: geometry collision mesh filename=../meshes/thumb_knuckle.obj; visual mesh filename=../meshes/thumb_knuckle.obj
- link right_thumb_swivel_link: geometry visual mesh filename=../meshes/thumb_swivel_link.obj
